Commit message: world base book rrbot

File: test_robot/urdf/rrbot.xacro (robot description, xacro)
@@ -17,33 +17,33 @@
   </gazebo>
   <!-- Link3 -->
-  <gazebo reference="link3">
+   <gazebo reference="link3">
     <mu1>0.2</mu1>
     <mu2>0.2</mu2>
     <material>Gazebo/Orange</material>
-  </gazebo>
-  <material name="black">
+       </gazebo>
+    <material name="black">
     <color rgba="0.0 0.0 0.0 1.0"/>
-  </material>
-  <material name="blue">
+   </material>
+   <material name="blue">
     <color rgba="0.0 0.0 0.8 1.0"/>
-  </material>
-  <material name="green">
-    <color rgba="0.0 0.8 0.0 1.0"/>
-  </material>
-  <material name="grey">
-    <color rgba="0.2 0.2 0.2 1.0"/>
-  </material>
-  <material name="orange">
-    <color rgba="1.0 0.423529411765 0.0392156862745 1.0"/>
-  </material>
-  <material name="brown">
-    <color rgba="0.870588235294 0.811764705882 0.764705882353 1.0"/>
-  </material>
-  <material name="red">
-    <color rgba="0.8 0.0 0.0 1.0"/>
-  </material>
-  <material name="white">
-    <color rgba="1.0 1.0 1.0 1.0"/>
-  </material>
+    </material>
+    <material name="green">
+      <color rgba="0.0 0.8 0.0 1.0"/>
+    </material>
+    <material name="grey">
+      <color rgba="0.2 0.2 0.2 1.0"/>
+    </material>
+    <material name="orange">
+      <color rgba="1.0 0.423529411765 0.0392156862745 1.0"/>
+    </material>
+    <material name="brown">
+      <color rgba="0.870588235294 0.811764705882 0.764705882353 1.0"/>
+    </material>
+    <material name="red">
+      <color rgba="0.8 0.0 0.0 1.0"/>
+    </material>
+    <material name="white">
+      <color rgba="1.0 1.0 1.0 1.0"/>
+    </material>
   <!-- Used for fixing robot to Gazebo 'base_link' -->
   <link name="world"/>

File: test_robot/urdf/rrbotbook.xacro (robot description, xacro)
@@ -13,6 +13,12 @@
      </inertial>
      </xacro:macro>
+  <link name="world"/>
+  <joint name="fixed" type="fixed">
+    <parent link="world"/>
+    <child link="base_link"/>
+  </joint>
  <!-- Base Link -->
    <link name="base_link">
+   <parent link="world" />
     <visual>
      <origin xyz="0 0 ${height1/2}" rpy="0 0 0" />
