Commit message: updates to inertia

File: test_robot/urdf/rrbotbook.xacro (robot description, xacro)
@@ -5,6 +5,12 @@
     <xacro:property name="height3" value="1" />
     <xacro:property name="axle_offset" value="0.05" />
-     <xacro:property name="damp" value="0.7" />
-  <!-- Base Link -->
+    <xacro:property name="damp" value="0.7" />
+ <xacro:macro name="default_inertial" params="z_value i_value  mass">
+    <inertial>
+    <origin xyz="0 0 ${z_value}" rpy="0 0 0"/>
+     <mass value="${mass}" />
+     <inertia ixx="${i_value}" ixy="0.0" ixz="0.0"        iyy="${i_value}" iyz="0.0"        izz="${i_value}" />
+     </inertial>  </xacro:macro>
+ <!-- Base Link -->
    <link name="base_link">
     <visual>
@@ -21,4 +27,5 @@
                         </collision>
                         <inertial>
+                         <xacro:default_inertial z_value="${computation for <origin> in    z-axis}" i_value="1.0" mass="1"/>
                          <origin xyz="0 0 ${height1/2}" rpy="0 0 0" />
                             <mass value="1" />
@@ -50,4 +57,5 @@
                    </collision>
                     <inertial>
+                     <xacro:default_inertial z_value="${computation for <origin> in    z-axis}" i_value="1.0" mass="1"/>
                       <origin xyz="0 0 ${height2/2 - axle_offset}" rpy="0 0 0" />
                            <mass value="1" />
@@ -79,8 +87,10 @@
                                   </collision>
                                     <inertial>
+                                     <xacro:default_inertial z_value="${computation for <origin> in    z-axis}" i_value="1.0" mass="1"/>
                                        <origin xyz="0 0 ${height3/2 - axle_offset}" rpy="0 0 0" />
                                           <mass value="1" />
                                           <inertia ixx="1.0" ixy="0.0" ixz="0.0" iyy="1.0" iyz="0.0"  izz="1.0" />
                                              </inertial>
+                                              <xacro:default_inertial z_value="${computation for <origin> in    z-axis}" i_value="1.0" mass="1"/>
                                                </link>
                                                 </robot>

Commit message: materials update for rrbot2

File: test_robot/urdf/rrbotbook.xacro (robot description, xacro)
@@ -11,5 +11,6 @@
      <mass value="${mass}" />
      <inertia ixx="${i_value}" ixy="0.0" ixz="0.0"        iyy="${i_value}" iyz="0.0"        izz="${i_value}" />
-     </inertial>  </xacro:macro>
+     </inertial>
+     </xacro:macro>
  <!-- Base Link -->
    <link name="base_link">

Commit message: rrbot book

File: test_robot/urdf/rrbotbook.xacro (robot description, xacro)
@@ -13,12 +13,11 @@
      </inertial>
      </xacro:macro>
-  <link name="world"/>
-  <joint name="fixed" type="fixed">
+<link name="world"/>
+<joint name="fixed" type="fixed">
     <parent link="world"/>
     <child link="base_link"/>
-  </joint>
+</joint>
  <!-- Base Link -->
    <link name="base_link">
-   <parent link="world" />
     <visual>
      <origin xyz="0 0 ${height1/2}" rpy="0 0 0" />
