Commit message: mesh for grippers

File: test_robot/urdf/materials.xacro (robot description, xacro)
@@ -4,23 +4,23 @@
  <color rgba="0.0 0.0 0.0 1.0"/>
  </material>
-  <material name="blue">
+<material name="blue">
   <color rgba="0.0 0.0 0.8 1.0"/>
   </material>
-  <material name="green">
+ <material name="green">
   <color rgba="0.0 1.0 0.0 1.0"/>
   </material>
-  <material name="grey">
+<material name="grey">
   <color rgba="0.2 0.2 0.2 1.0"/>
   </material>
-  <material name="orange">
+   <material name="orange">
   <color rgba="${255/255} ${108/255} ${10/255} 1.0"/>
   </material>
-  <material name="brown">
+ <material name="brown">
   <color rgba="${222/255} ${207/255} ${195/255} 1.0"/>
   </material>
-  <material name="red">
+ <material name="red">
   <color rgba="0.8 0.0 0.0 1.0"/>
   </material>
-  <material name="white">
+ <material name="white">
   <color rgba="1.0 1.0 1.0 1.0"/>
   </material>

File: test_robot/urdf/rrbot2.xacro (robot description, xacro)
@@ -8,5 +8,5 @@
  <!-- Import Rviz colors -->
  <xacro:include
- filename="$(find ros_robotics)/urdf/materials.xacro" />
+ filename="$(find test_robot)/urdf/materials.xacro" />
   <!-- Default Inertial -->
   <xacro:macro name="default_inertial" params="z_value i_value mass">
