Commit message: testing

File: test_robot/urdf/rrbot2.xacro (robot description, xacro)
@@ -1,30 +1,111 @@
-<?xml version="1.0"?>
+<?xml version="1.0" ?>
+<!-- =================================================================================== -->
+<!-- |    This document was autogenerated by xacro from rrbot.xacro                    | -->
+<!-- |    EDITING THIS FILE BY HAND IS NOT RECOMMENDED                                 | -->
+<!-- =================================================================================== -->
 <!-- Revolute-Revolute Manipulator -->
-…
-  <!-- Import Rviz colors -->
-  <xacro:include            filename="$(find test_robot)/urdf/materials.xacro" />
-  <!-- Default Inertial -->
-  <xacro:macro name="default_inertial" params="z_value i_value mass">
-  <inertial>
-  <origin xyz="0 0 ${z_value}" rpy="0 0 0"/>
-  <mass value="${mass}" />
-  <inertia ixx="${i_value}" ixy="0.0" ixz="0.0"               iyy="${i_value}" iyz="0.0"
-   izz="${i_value}" />
-   </inertial>
-   </xacro:macro>
+<robot name="rrbot" xmlns:xacro="http://www.ros.org/wiki/xacro">
+ <!-- Used for fixing robot to Gazebo 'base_link' -->
+  <link name="world"/>
+  <joint name="fixed" type="fixed">
+    <parent link="world"/>
+    <child link="link1"/>
+  </joint>
   <!-- Base Link -->
-  …
-  </collision>
-    <xacro:default_inertial z_value="${height1/2}"
-                i_value="1.0" mass="1"/>  </link>
-                …
-     <!-- Middle Link -->
-                 …
-                 </collision>
-        <xacro:default_inertial z_value="${height2/2 - axle_offset}"  i_value="1.0" mass="1"/>
-       </link>
-         …
-    <!-- Top Link -->    …    </collision>
-    <xacro:default_inertial z_value="${height3/2 - axle_offset}"      i_value="1.0" mass="1"/>
-      </link>
+  <link name="link1">
+    <collision>
+      <origin rpy="0 0 0" xyz="0 0 1.0"/>
+      <geometry>
+        <box size="0.1 0.1 2"/>
+      </geometry>
+    </collision>
+    <visual>
+      <origin rpy="0 0 0" xyz="0 0 1.0"/>
+      <geometry>
+        <box size="0.1 0.1 2"/>
+      </geometry>
+      <material name="orange"/>
+    </visual>
+    <inertial>
+      <origin rpy="0 0 0" xyz="0 0 1.0"/>
+      <mass value="1"/>
+      <inertia ixx="0.334166666667" ixy="0.0" ixz="0.0" iyy="0.334166666667" iyz="0.0" izz="0.00166666666667"/>
+    </inertial>
+  </link>
+  <joint name="joint1" type="continuous">
+    <parent link="link1"/>
+    <child link="link2"/>
+    <origin rpy="0 0 0" xyz="0 0.1 1.95"/>
+    <axis xyz="0 1 0"/>
+    <dynamics damping="0.7"/>
+  </joint>
+  <!-- Middle Link -->
+  <link name="link2">
+    <collision>
+      <origin rpy="0 0 0" xyz="0 0 0.45"/>
+      <geometry>
+        <box size="0.1 0.1 1"/>
+      </geometry>
+    </collision>
+    <visual>
+      <origin rpy="0 0 0" xyz="0 0 0.45"/>
+      <geometry>
+        <box size="0.1 0.1 1"/>
+      </geometry>
+      <material name="black"/>
+    </visual>
+    <inertial>
+      <origin rpy="0 0 0" xyz="0 0 0.45"/>
+      <mass value="1"/>
+      <inertia ixx="0.0841666666667" ixy="0.0" ixz="0.0" iyy="0.0841666666667" iyz="0.0" izz="0.00166666666667"/>
+    </inertial>
+  </link>
+  <joint name="joint2" type="continuous">
+    <parent link="link2"/>
+    <child link="link3"/>
+    <origin rpy="0 0 0" xyz="0 0.1 0.9"/>
+    <axis xyz="0 1 0"/>
+    <dynamics damping="0.7"/>
+  </joint>
+  <!-- Top Link -->
+  <link name="link3">
+    <collision>
+      <origin rpy="0 0 0" xyz="0 0 0.45"/>
+      <geometry>
+        <box size="0.1 0.1 1"/>
+      </geometry>
+    </collision>
+    <visual>
+      <origin rpy="0 0 0" xyz="0 0 0.45"/>
+      <geometry>
+        <box size="0.1 0.1 1"/>
+      </geometry>
+      <material name="orange"/>
+    </visual>
+    <inertial>
+      <origin rpy="0 0 0" xyz="0 0 0.45"/>
+      <mass value="1"/>
+      <inertia ixx="0.0841666666667" ixy="0.0" ixz="0.0" iyy="0.0841666666667" iyz="0.0" izz="0.00166666666667"/>
+    </inertial>
+  </link>
+  <transmission name="tran1">
+    <type>transmission_interface/SimpleTransmission</type>
+    <joint name="joint1">
+      <hardwareInterface>hardware_interface/EffortJointInterface</hardwareInterface>
+    </joint>
+    <actuator name="motor1">
+      <hardwareInterface>hardware_interface/EffortJointInterface</hardwareInterface>
+      <mechanicalReduction>1</mechanicalReduction>
+    </actuator>
+  </transmission>
+  <transmission name="tran2">
+    <type>transmission_interface/SimpleTransmission</type>
+    <joint name="joint2">
+      <hardwareInterface>hardware_interface/EffortJointInterface</hardwareInterface>
+    </joint>
+    <actuator name="motor2">
+      <hardwareInterface>hardware_interface/EffortJointInterface</hardwareInterface>
+      <mechanicalReduction>1</mechanicalReduction>
+    </actuator>
+  </transmission>
 </robot>

Commit message: rrbot 2

File: test_robot/urdf/rrbot2.xacro (robot description, xacro)
@@ -6,4 +6,15 @@
 <!-- Revolute-Revolute Manipulator -->
 <robot name="rrbot" xmlns:xacro="http://www.ros.org/wiki/xacro">
+ <!-- Import Rviz colors -->
+ <xacro:include
+ filename="$(find ros_robotics)/urdf/materials.xacro" />
+  <!-- Default Inertial -->
+  <xacro:macro name="default_inertial" params="z_value i_value mass">
+  <inertial>
+  <origin xyz="0 0 ${z_value}" rpy="0 0 0"/>
+  <mass value="${mass}" />
+  <inertia ixx="${i_value}" ixy="0.0" ixz="0.0"               iyy="${i_value}" iyz="0.0"  izz="${i_value}" />
+   </inertial>
+   </xacro:macro>
  <!-- Used for fixing robot to Gazebo 'base_link' -->
   <link name="world"/>
@@ -20,4 +31,6 @@
       </geometry>
     </collision>
+    <xacro:default_inertial z_value="${height1/2}"
+                 i_value="1.0" mass="1"/>
     <visual>
       <origin rpy="0 0 0" xyz="0 0 1.0"/>
@@ -48,4 +61,5 @@
       </geometry>
     </collision>
+     <xacro:default_inertial z_value="${height2/2 - axle_offset}"    i_value="1.0" mass="1"/>
     <visual>
       <origin rpy="0 0 0" xyz="0 0 0.45"/>
@@ -76,4 +90,5 @@
       </geometry>
     </collision>
+        <xacro:default_inertial z_value="${height3/2 - axle_offset}"      i_value="1.0" mass="1"/>
     <visual>
       <origin rpy="0 0 0" xyz="0 0 0.45"/>

Commit message: rrbot3 setup

File: test_robot/urdf/rrbot2.xacro (robot description, xacro)
@@ -38,5 +38,5 @@
         <box size="0.1 0.1 2"/>
       </geometry>
-      <material name="orange"/>
+      <material name="blue"/>
     </visual>
     <inertial>
@@ -67,5 +67,5 @@
         <box size="0.1 0.1 1"/>
       </geometry>
-      <material name="black"/>
+      <material name="red"/>
     </visual>
     <inertial>
@@ -96,5 +96,5 @@
         <box size="0.1 0.1 1"/>
       </geometry>
-      <material name="orange"/>
+      <material name="green"/>
     </visual>
     <inertial>

File: test_robot/urdf/rrbot3.xacro (robot description, xacro)
@@ -7,6 +7,7 @@
 <robot name="rrbot" xmlns:xacro="http://www.ros.org/wiki/xacro">
  <!-- Import Rviz colors -->
- <xacro:include            filename="$(find test_robot)/urdf/materials.xacro" />
- <xacro:include filename="$(find test_robot)/urdf/gripper.xacro" /
+ <xacro:include filename="$(find test_robot)/urdf/materials.xacro" />
+ <!--Include gripper files-->>
+ <xacro:include filename="$(find test_robot)/urdf/gripper.xacro" />
   <!-- Default Inertial -->
   <xacro:macro name="default_inertial" params="z_value i_value mass">
@@ -104,4 +105,12 @@
     </inertial>
   </link>
+  <!-- Gripper Link -->>
+  <link name="left_gripper">
+    <visual>
+    <origin rpy="0 0 0" xyz="0 0 0"/>
+    <geometry>
+    <mesh filename="package://pr2_common/meshes/l_finger.dae"/>
+        </geometry>
+        </visual>
   <transmission name="tran1">
     <type>transmission_interface/SimpleTransmission</type>

Commit message: color

File: test_robot/urdf/rrbot2.xacro (robot description, xacro)
@@ -34,9 +34,9 @@
                  i_value="1.0" mass="1"/>
     <visual>
+     <material name="blue"/>
       <origin rpy="0 0 0" xyz="0 0 1.0"/>
       <geometry>
         <box size="0.1 0.1 2"/>
       </geometry>
-      <material name="blue"/>
     </visual>
     <inertial>
