Commit message: repo

File: test_robot/urdf/gripper.xacro (robot description, xacro)
@@ -12,5 +12,5 @@
   <origin rpy="0 0 0" xyz="0 0 0"/>
   <geometry>
-  <mesh filename="package://pr2_common/meshes/l_finger.dae"/>
+  <mesh filename="package://pr2_description/meshes/l_finger.dae"/>
   </geometry>
   </visual>
@@ -29,5 +29,5 @@
   <origin rpy="0 0 0" xyz="0.09137 0.00495 0"/>
   <geometry>
-  <mesh           filename="package://pr2_common/meshes/l_finger_tip.dae"/>
+  <mesh           filename="package://pr2_description/meshes/l_finger_tip.dae"/>
   </geometry>
    </visual>
@@ -50,5 +50,5 @@
   <origin rpy="3.1415 0 0" xyz="0 0 0"/>
    <geometry>
-   <mesh filename="package://pr2_common/meshes/l_finger.dae"/>
+   <mesh filename="package://pr2_description/meshes/l_finger.dae"/>
    </geometry>
    </visual>
@@ -68,5 +68,5 @@
    <origin rpy="-3.1415 0 0" xyz="0.09137 0.00495 0"/>
    <geometry>
-   <mesh           filename="package://pr2_common/meshes/l_finger_tip.dae"/>
+   <mesh           filename="package://pr2_description/meshes/l_finger_tip.dae"/>
    </geometry>
    </visual>

File: test_robot/urdf/rrbot3.xacro (robot description, xacro)
@@ -110,5 +110,5 @@
     <origin rpy="0 0 0" xyz="0 0 0"/>
     <geometry>
-    <mesh filename="package://pr2_common/meshes/l_finger.dae"/>
+    <mesh filename="package://pr2_description/meshes/l_finger.dae"/>
         </geometry>
         </visual>
