Commit message: repo

File: test_robot/urdf/rrbot3.xacro (robot description, xacro)
@@ -106,11 +106,11 @@
   </link>
   <!-- Gripper Link -->>
-  <link name="left_gripper">
-    <visual>
-    <origin rpy="0 0 0" xyz="0 0 0"/>
-    <geometry>
-    <mesh filename="package://pr2_description/meshes/l_finger.dae"/>
-        </geometry>
-        </visual>
+    <link name="left_gripper">
+      <visual>
+      <origin rpy="0 0 0" xyz="0 0 0"/>
+      <geometry>
+      <mesh filename="package://pr2_common/meshes/l_finger.dae"/>
+          </geometry>
+          </visual>
   <transmission name="tran1">
     <type>transmission_interface/SimpleTransmission</type>

Commit message: repo description

File: test_robot/urdf/rrbot3.xacro (robot description, xacro)
@@ -110,5 +110,5 @@
       <origin rpy="0 0 0" xyz="0 0 0"/>
       <geometry>
-      <mesh filename="package://pr2_common/meshes/l_finger.dae"/>
+      <mesh filename="package://pr2_description/meshes/l_finger.dae"/>
           </geometry>
           </visual>
